File: Version 1/Hardware/E-CAD/WDM(RevB_V1).kicad_pcb (KiCad board)
At the start: 4 copper layers, 61 x 68.8 mm, 114 parts, among them J11 SJ-3542AS-SMT-TR-67, J14 CONN HEADER SMD R/A 2POS 1.25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, J15 SJ-3541AS-SMT-TR-67, J2 T4.1, J3 SJ-3542AS-SMT-TR-67, J6 SJ-3542AS-SMT-TR-67, J7 SJ-3542AS-SMT-TR-67, SW1 JS202011JAQN Slide Switch DPD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, T1 MMUN2133LT1G, U1 TPS61090RSAR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

Commit message: Updated PCB zones & board outline. Also  uploaded revised pin definitions to match routing
Connections:
- J2 pad GND_0: unconnected-(J2-PadGND_0) -> GND
- J2 pad GND_1: unconnected-(J2-PadGND_1) -> GND
- J2 pad GND_2: unconnected-(J2-PadGND_2) -> GND
Other:
- outline, holes or cut-outs redrawn
